Commit message: 完成了x = [z, phi, theta, varphi1..varphi6]^T的形式

File: Go2Arm_description/urdf/vis_piper_description_mjc_NoGripper.urdf (robot description, URDF)
Before this commit: robot piperNoGripper_description, 9 links, 8 joints
Links:
- added link base_roll, mass 1e-3
- added link base_z, mass 1e-3
- added link world
Joints:
- added joint root_pitch: type revolute, parent base_roll, child base, origin xyz=0 0 0 rpy=0 0 0, axis 0 1 0, limit lower=-1.57 upper=1.57 effort=1000 velocity=3.0
- added joint root_roll: type revolute, parent base_z, child base_roll, origin xyz=0 0 0 rpy=0 0 0, axis 1 0 0, limit lower=-1.57 upper=1.57 effort=1000 velocity=3.0
- added joint root_z: type prismatic, parent world, child base_z, origin xyz=0 0 0 rpy=0 0 0, axis 0 0 1, limit lower=0.0 upper=1.0 effort=1000 velocity=2.0
